Commit message: quad_control_gz: modify joint name in anymal urdf for duplicated name issue

File: quad_control_gz/urdf/anymal.urdf (robot description, URDF)
Before this commit: robot anymal, 78 links, 77 joints
Joints:
- removed joint LF_HAA
- removed joint LF_HFE
- removed joint LF_KFE
- removed joint LH_HAA
- removed joint LH_HFE
- removed joint LH_KFE
- removed joint RF_HAA
- removed joint RF_HFE
- removed joint RF_KFE
- removed joint RH_HAA
- removed joint RH_HFE
- removed joint RH_KFE
- added joint LF_HAA_LF_HIP: type revolute, parent LF_HAA, child LF_HIP, origin xyz=0 0 0 rpy=0 0 0, axis 1 0 0, limit lower=-0.72 upper=0.49 effort=80.0 velocity=7.5
- added joint LF_HFE_LF_THIGH: type revolute, parent LF_HFE, child LF_THIGH, origin xyz=0 0 0 rpy=0 0 0, axis 1 0 0, limit lower=-9.42477796077 upper=9.42477796077 effort=80.0 velocity=7.5
- added joint LF_KFE_LF_SHANK: type revolute, parent LF_KFE, child LF_SHANK, origin xyz=0 0 0 rpy=0 0 0, axis 1 0 0, limit lower=-9.42477796077 upper=9.42477796077 effort=80.0 velocity=7.5
- added joint LH_HAA_LH_HIP: type revolute, parent LH_HAA, child LH_HIP, origin xyz=0 0 0 rpy=0 0 0, axis -1 0 0, limit lower=-0.72 upper=0.49 effort=80.0 velocity=7.5
- added joint LH_HFE_LH_THIGH: type revolute, parent LH_HFE, child LH_THIGH, origin xyz=0 0 0 rpy=0 0 0, axis 1 0 0, limit lower=-9.42477796077 upper=9.42477796077 effort=80.0 velocity=7.5
- added joint LH_KFE_LH_SHANK: type revolute, parent LH_KFE, child LH_SHANK, origin xyz=0 0 0 rpy=0 0 0, axis 1 0 0, limit lower=-9.42477796077 upper=9.42477796077 effort=80.0 velocity=7.5
- added joint RF_HAA_RF_HIP: type revolute, parent RF_HAA, child RF_HIP, origin xyz=0 0 0 rpy=0 0 0, axis 1 0 0, limit lower=-0.49 upper=0.72 effort=80.0 velocity=7.5
- added joint RF_HFE_RF_THIGH: type revolute, parent RF_HFE, child RF_THIGH, origin xyz=0 0 0 rpy=0 0 0, axis -1 0 0, limit lower=-9.42477796077 upper=9.42477796077 effort=80.0 velocity=7.5
- added joint RF_KFE_RF_SHANK: type revolute, parent RF_KFE, child RF_SHANK, origin xyz=0 0 0 rpy=0 0 0, axis -1 0 0, limit lower=-9.42477796077 upper=9.42477796077 effort=80.0 velocity=7.5
- added joint RH_HAA_RH_HIP: type revolute, parent RH_HAA, child RH_HIP, origin xyz=0 0 0 rpy=0 0 0, axis -1 0 0, limit lower=-0.49 upper=0.72 effort=80.0 velocity=7.5
- added joint RH_HFE_RH_THIGH: type revolute, parent RH_HFE, child RH_THIGH, origin xyz=0 0 0 rpy=0 0 0, axis -1 0 0, limit lower=-9.42477796077 upper=9.42477796077 effort=80.0 velocity=7.5
- added joint RH_KFE_RH_SHANK: type revolute, parent RH_KFE, child RH_SHANK, origin xyz=0 0 0 rpy=0 0 0, axis -1 0 0, limit lower=-9.42477796077 upper=9.42477796077 effort=80.0 velocity=7.5
