Commit message: quad_control_gz: register imu

File: quad_control_gz/urdf/anymal.gazebo.xacro (robot description, xacro)
@@ -4,4 +4,6 @@
         <plugin filename="gz_ros2_control-system" name="gz_ros2_control::GazeboSimROS2ControlPlugin">
         <parameters>$(find quad_control_gz)/config/config.yaml</parameters>
+        </plugin>
+        <plugin filename="gz-sim-imu-system" name="gz::sim::systems::Imu">
         </plugin>
     </gazebo>
@@ -16,3 +18,9 @@
     <xacro:preserve_fixed_joint joint_name="LH_shank_fixed_LH_FOOT"/>
     <xacro:preserve_fixed_joint joint_name="RH_shank_fixed_RH_FOOT"/>
+    <gazebo reference="imu_link">
+        <sensor name="base_imu" type="imu">
+            <always_on>1</always_on>
+            <update_rate>500</update_rate>
+        </sensor>
+    </gazebo>
 </robot>

File: quad_control_gz/urdf/anymal.ros2_control.xacro (robot description, xacro)
@@ -40,4 +40,21 @@
             <state_interface name="linear_acceleration.y"/>
             <state_interface name="linear_acceleration.z"/>
+            <xacro:macro name="covariance_generator" params="prefix">
+                <state_interface name="${prefix}.xx"/>
+                <state_interface name="${prefix}.xy"/>
+                <state_interface name="${prefix}.xz"/>
+                <state_interface name="${prefix}.yx"/>
+                <state_interface name="${prefix}.yy"/>
+                <state_interface name="${prefix}.yz"/>
+                <state_interface name="${prefix}.zx"/>
+                <state_interface name="${prefix}.zy"/>
+                <state_interface name="${prefix}.zz"/>
+            </xacro:macro>
+            <xacro:covariance_generator prefix="orientation_covariance"/>
+            <xacro:covariance_generator prefix="angular_velocity_covariance"/>
+            <xacro:covariance_generator prefix="linear_acceleration_covariance"/>
+            <param name="orientation_covariance_diagonal">0.0012</param>
+            <param name="angular_velocity_covariance_diagonal">0.0004</param>
+            <param name="linear_acceleration_covariance_diagonal">0.01</param>
         </sensor>
         <sensor name="LF_FOOT_sensor"><state_interface name="contact"/></sensor>

Commit message: quad_control_gz: setup ft interface in urdf:

File: quad_control_gz/urdf/anymal.gazebo.xacro (robot description, xacro)
@@ -6,4 +6,6 @@
         </plugin>
         <plugin filename="gz-sim-imu-system" name="gz::sim::systems::Imu">
+        </plugin>
+        <plugin filename="gz-sim-force-torque-system" name="gz::sim::systems::ForceTorque">
         </plugin>
     </gazebo>
@@ -23,5 +25,24 @@
             <update_rate>500</update_rate>
             <topic>imu</topic>
+            <visualize>true</visualize>
         </sensor>
     </gazebo>
+    <xacro:macro name="foot_ft" params="prefix">
+        <gazebo reference="${prefix}_FOOT">
+        <sensor name="${prefix}_ft" type="force_torque">
+            <always_on>true</always_on>
+            <update_rate>500</update_rate>
+            <topic>${prefix}/ft</topic>
+            <visualize>true</visualize>
+            <force_torque>
+                <frame>child</frame>
+                <measure_direction>child_to_parent</measure_direction>
+            </force_torque>
+        </sensor>
+        </gazebo>
+    </xacro:macro>
+    <xacro:foot_ft prefix="LF"/>
+    <xacro:foot_ft prefix="RF"/>
+    <xacro:foot_ft prefix="LH"/>
+    <xacro:foot_ft prefix="RH"/>
 </robot>

File: quad_control_gz/urdf/anymal.ros2_control.xacro (robot description, xacro)
@@ -62,4 +62,13 @@
         <sensor name="LH_FOOT_sensor"><state_interface name="contact"/></sensor>
         <sensor name="RH_FOOT_sensor"><state_interface name="contact"/></sensor>
+        <xacro:macro name="foot_contact_interface" params="prefix">
+            <sensor name="${prefix}_ft">
+            <state_interface name="contact"/>
+            </sensor>
+        </xacro:macro>
+        <xacro:foot_contact_interface prefix="LF"/>
+        <xacro:foot_contact_interface prefix="RF"/>
+        <xacro:foot_contact_interface prefix="LH"/>
+        <xacro:foot_contact_interface prefix="RH"/>
     </ros2_control>
 </robot>
