Commit message: quad_control: sync urdf and joint names

File: quad_control_gz/urdf/anymal.complete.xacro (robot description, xacro)
@@ -1,5 +1,5 @@
 <?xml version="1.0"?>
 <robot xmlns:xacro="http://www.ros.org" name="anymal">
-    <xacro:include filename="$(find quad_control_gz)/urdf/anymal.urdf" />
+    <xacro:include filename="$(find quad_control_gz)/urdf/anymal_c/urdf/anymal.urdf" />
     <xacro:include filename="$(find quad_control_gz)/urdf/anymal.gazebo.xacro" />
     <xacro:include filename="$(find quad_control_gz)/urdf/anymal.ros2_control.xacro" />

File: quad_control_gz/urdf/anymal.gazebo.xacro (robot description, xacro)
@@ -11,9 +11,9 @@
         <plugin filename="gz-sim-odometry-publisher-system" name="gz::sim::systems::OdometryPublisher">
             <odom_topic>/ground_truth/state</odom_topic>
-            <tf_topic>/tf</tf_topic>
-            <odom_frame>world</odom_frame>
-            <robot_base_frame>base</robot_base_frame>
             <dimensions>3</dimensions>
             <update_rate>500</update_rate>
+            <!-- <tf_topic>/tf</tf_topic>
+            <odom_frame>odom</odom_frame>
+            <robot_base_frame>base</robot_base_frame> -->
         </plugin>
     </gazebo>

File: quad_control_gz/urdf/anymal_c/urdf/anymal.urdf (robot description, URDF)
Before this commit: robot anymal, 78 links, 77 joints
Links:
- link LF_FOOT: geometry collision cylinder length=0.282504 radius=0.0175; collision sphere radius=0.03
- link LF_HAA: geometry visual mesh filename=package://quad_control_gz/urdf/anymal_c/meshes/drive.dae scale=1.0 1.0 1.0
- link LF_HFE: geometry collision cylinder length=0.14 radius=0.05; visual mesh filename=package://quad_control_gz/urdf/anymal_c/meshes/drive.dae scale=1.0 1.0 1.0
- link LF_KFE: geometry collision cylinder length=0.14 radius=0.05; visual mesh filename=package://quad_control_gz/urdf/anymal_c/meshes/drive.dae scale=1.0 1.0 1.0
- link LF_hip_fixed: geometry visual mesh filename=package://quad_control_gz/urdf/anymal_c/meshes/hip_l.dae scale=1.0 1.0 1.0
- link LF_shank_fixed: geometry collision box size=0.114998 0.0675 0.04; collision cylinder length=0.04 radius=0.06
- link LF_thigh_fixed: geometry collision box size=0.075 0.06 0.282627; collision cylinder length=0.08 radius=0.065
- link LH_FOOT: geometry collision cylinder length=0.282504 radius=0.0175; collision sphere radius=0.03
- link LH_HAA: geometry visual mesh filename=package://quad_control_gz/urdf/anymal_c/meshes/drive.dae scale=1.0 1.0 1.0
- link LH_HFE: geometry collision cylinder length=0.14 radius=0.05; visual mesh filename=package://quad_control_gz/urdf/anymal_c/meshes/drive.dae scale=1.0 1.0 1.0
- link LH_KFE: geometry collision cylinder length=0.14 radius=0.05; visual mesh filename=package://quad_control_gz/urdf/anymal_c/meshes/drive.dae scale=1.0 1.0 1.0
- link LH_hip_fixed: geometry visual mesh filename=package://quad_control_gz/urdf/anymal_c/meshes/hip_r.dae scale=1.0 1.0 1.0
- link LH_shank_fixed: geometry collision box size=0.114998 0.0675 0.04; collision cylinder length=0.04 radius=0.06
- link LH_thigh_fixed: geometry collision box size=0.075 0.06 0.282627; collision cylinder length=0.08 radius=0.065
- link RF_FOOT: geometry collision cylinder length=0.282504 radius=0.0175; collision sphere radius=0.03
- link RF_HAA: geometry visual mesh filename=package://quad_control_gz/urdf/anymal_c/meshes/drive.dae scale=1.0 1.0 1.0
- link RF_HFE: geometry collision cylinder length=0.14 radius=0.05; visual mesh filename=package://quad_control_gz/urdf/anymal_c/meshes/drive.dae scale=1.0 1.0 1.0
- link RF_KFE: geometry collision cylinder length=0.14 radius=0.05; visual mesh filename=package://quad_control_gz/urdf/anymal_c/meshes/drive.dae scale=1.0 1.0 1.0
- link RF_hip_fixed: geometry visual mesh filename=package://quad_control_gz/urdf/anymal_c/meshes/hip_r.dae scale=1.0 1.0 1.0
- link RF_shank_fixed: geometry collision box size=0.114998 0.0675 0.04; collision cylinder length=0.04 radius=0.06
- link RF_thigh_fixed: geometry collision box size=0.075 0.06 0.282627; collision cylinder length=0.08 radius=0.065
- link RH_FOOT: geometry collision cylinder length=0.282504 radius=0.0175; collision sphere radius=0.03
- link RH_HAA: geometry visual mesh filename=package://quad_control_gz/urdf/anymal_c/meshes/drive.dae scale=1.0 1.0 1.0
- link RH_HFE: geometry collision cylinder length=0.14 radius=0.05; visual mesh filename=package://quad_control_gz/urdf/anymal_c/meshes/drive.dae scale=1.0 1.0 1.0
- link RH_KFE: geometry collision cylinder length=0.14 radius=0.05; visual mesh filename=package://quad_control_gz/urdf/anymal_c/meshes/drive.dae scale=1.0 1.0 1.0
- link RH_hip_fixed: geometry visual mesh filename=package://quad_control_gz/urdf/anymal_c/meshes/hip_l.dae scale=1.0 1.0 1.0
- link RH_shank_fixed: geometry collision box size=0.114998 0.0675 0.04; collision cylinder length=0.04 radius=0.06
- link RH_thigh_fixed: geometry collision box size=0.075 0.06 0.282627; collision cylinder length=0.08 radius=0.065
- link base: geometry collision box size=0.58 0.14 0.18; collision cylinder length=0.145 radius=0.09
- link battery: geometry visual mesh filename=package://quad_control_gz/urdf/anymal_c/meshes/battery.dae scale=1.0 1.0 1.0
- link bottom_shell: geometry visual mesh filename=package://quad_control_gz/urdf/anymal_c/meshes/bottom_shell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 scale=1.0 1.0 1.0
- link depth_camera_front_camera: geometry visual mesh filename=package://quad_control_gz/urdf/anymal_c/meshes/depth_camera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 scale=1.0 1.0 1.0
- link depth_camera_left_camera: geometry visual mesh filename=package://quad_control_gz/urdf/anymal_c/meshes/depth_camera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 scale=1.0 1.0 1.0
- link depth_camera_rear_camera: geometry visual mesh filename=package://quad_control_gz/urdf/anymal_c/meshes/depth_camera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 scale=1.0 1.0 1.0
- link depth_camera_right_camera: geometry visual mesh filename=package://quad_control_gz/urdf/anymal_c/meshes/depth_camera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 scale=1.0 1.0 1.0
- link face_front: geometry collision box size=0.11 0.14 0.18; collision cylinder length=0.11 radius=0.09
- link face_rear: geometry collision box size=0.11 0.14 0.18; collision cylinder length=0.11 radius=0.09
- link handle: geometry visual mesh filename=package://quad_control_gz/urdf/anymal_c/meshes/handle.dae scale=1.0 1.0 1.0
- link hatch: geometry visual mesh filename=package://quad_control_gz/urdf/anymal_c/meshes/hatch.dae scale=1.0 1.0 1.0
- link lidar: geometry visual mesh filename=package://quad_control_gz/urdf/anymal_c/meshes/lidar.dae
- link lidar_cage: geometry collision cylinder length=0.12 radius=0.07; visual mesh filename=package://quad_control_gz/urdf/anymal_c/meshes/lidar_cage.d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 scale=1.0 1.0 1.0
- link remote: geometry visual mesh filename=package://quad_control_gz/urdf/anymal_c/meshes/remote.dae scale=1.0 1.0 1.0
- link top_shell: geometry visual mesh filename=package://quad_control_gz/urdf/anymal_c/meshes/top_shell.dae scale=1.0 1.0 1.0
- link wide_angle_camera_front_camera: geometry visual mesh filename=package://quad_control_gz/urdf/anymal_c/meshes/wide_angle_c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 scale=1.0 1.0 1.0
- link wide_angle_camera_rear_camera: geometry visual mesh filename=package://quad_control_gz/urdf/anymal_c/meshes/wide_angle_c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 scale=1.0 1.0 1.0
